Commit message: Add VAYRON ROS 2 control and hardware integration

File: src/vayron_description/urdf/vayron/vayron.urdf.xacro (robot description, xacro)
@@ -1,4 +1,6 @@
 <?xml version="1.0"?>
 <robot name="vayron" xmlns:xacro="http://www.ros.org/wiki/xacro">
+  <xacro:arg name="simulation" default="false"/>
+  <xacro:property name="simulation" value="$(arg simulation)"/>
   <xacro:property name="chassis_length" value="0.22"/>
   <xacro:property name="chassis_width" value="0.22"/>
@@ -127,6 +129,6 @@
     <origin xyz="0 0 0.006" rpy="0 0 0"/>
   </joint>
-  <!-- Arduino Mega -->
-  <link name="arduino_mega_link">
+  <!-- Arduino Uno -->
+  <link name="arduino_uno_link">
     <visual>
       <geometry>
@@ -136,7 +138,7 @@
     </visual>
   </link>
-  <joint name="arduino_mega_joint" type="fixed">
+  <joint name="arduino_uno_joint" type="fixed">
     <parent link="electronics_tray"/>
-    <child link="arduino_mega_link"/>
+    <child link="arduino_uno_link"/>
     <origin xyz="0.040 0 0.012" rpy="0 0 0"/>
   </joint>
@@ -272,5 +274,6 @@
   <xacro:ultrasonic name="ultrasonic_right_link" y="-0.050"/>
   <!-- Gazebo Classic simulated 360-degree LiDAR -->
-  <gazebo reference="rplidar_link">
+  <xacro:if value="$(arg simulation)">
+<gazebo reference="rplidar_link">
     <sensor name="vayron_lidar" type="ray">
       <pose>0 0 0 0 0 0</pose>
@@ -309,6 +312,8 @@
     </sensor>
   </gazebo>
+  </xacro:if>
   <!-- VAYRON differential drive controller for Gazebo Classic -->
-  <gazebo>
+  <xacro:if value="$(arg simulation)">
+<gazebo>
     <plugin name="vayron_diff_drive"
             filename="libgazebo_ros_diff_drive.so">
@@ -342,6 +347,8 @@
     </plugin>
   </gazebo>
+  </xacro:if>
   <!-- Publish actual Gazebo wheel joint states -->
-  <gazebo>
+  <xacro:if value="$(arg simulation)">
+<gazebo>
     <plugin name="gazebo_joint_state_publisher"
             filename="libgazebo_ros_joint_state_publisher.so">
@@ -357,3 +364,4 @@
     </plugin>
   </gazebo>
+  </xacro:if>
 </robot>
